Commit message: fix to correctly receive sensor data from gazebo

File: src/pandora_description/urdf/pandora.xacro (robot description, xacro)
@@ -76,5 +76,8 @@
 		<mass value="0.001"/>
 		<origin rpy="0 0 0" xyz="0 0 0"/>
-		<inertia ixx="0.0001" ixy="0" ixz="0" iyy="0.000001" iyz="0" izz="0.0001"/>
+		<inertia
+				  ixx="${0.001 / 12.0 * (0.001*0.001 + 0.001*0.001)}" ixy="0.0" ixz="0.0"
+				  iyy="${0.001 / 12.0 * (0.001*0.001 + 0.001*0.001)}" iyz="0.0"
+				  izz="${0.001 / 12.0 * (0.001*0.001 + 0.001*0.001)}"/>
 	</inertial>
 	<visual>
