Commit message: deleted old files, adjust .world files. MDH inverse kinematics is not working properly yet

File: src/pandora_description/urdf/leg.xacro (robot description, xacro)
@@ -22,5 +22,5 @@
 				<box size="${frame_x} ${frame_y} ${frame_z} "/>
 		  	</geometry>
-			<material name="blue">
+			<material name="Gazebo/blue">
 				<color rgba="0.0 0.0 0.8 1.0"/>
 			</material>
@@ -58,5 +58,5 @@
 				<box size="${crank_x} ${crank_y} ${crank_z} "/>
 		  	</geometry>
-			<material name="red">
+			<material name="Gazebo/Gazebo/red">
 				<color rgba="0.8 0.0 0.0 1.0"/>
 			</material>
@@ -93,5 +93,5 @@
 				<box size="${coupler_x} ${coupler_y} ${coupler_z} "/>
 		  	</geometry>
-			<material name="blue">
+			<material name="Gazebo/blue">
 				<color rgba="0.0 0.0 0.8 1.0"/>
 			</material>
@@ -128,5 +128,5 @@
 				<box size="${rocker_x} ${rocker_y} ${rocker_z}"/>
 		  	</geometry>
-			<material name="red">
+			<material name="Gazebo/red">
 				<color rgba="0.8 0.0 0.0 1.0"/>
 			</material>
@@ -273,6 +273,6 @@
 	</ros2_control>
 	<gazebo reference="my_box_link">
-		<material>Gazebo/Blue</material>
-		<material>Gazebo/Red</material>
+		<material>Gazebo/Gazebo/blue</material>
+		<material>Gazebo/Gazebo/red</material>
 	</gazebo>
 </xacro:macro>

File: src/pandora_description/urdf/pandora.xacro (robot description, xacro)
@@ -2,4 +2,5 @@
 <robot xmlns:xacro="http://www.ros.org/wiki/xacro" name="pandora">
 	<!-- other files -->
+	<xacro:include filename="$(find pandora_description)/materials.xacro" />
 	<xacro:include filename="$(find pandora_description)/urdf/parameters.xacro" />
 	<xacro:include filename="$(find pandora_description)/urdf/leg.xacro" />

File: src/pandora_description/urdf/parameters.xacro (robot description, xacro)
@@ -17,5 +17,5 @@
 	<xacro:property name="base_y" value="0.25" />		<!-- value in y axis -->
 	<xacro:property name="base_z" value="0.01" /> 	<!-- value in z axis -->
-	<xacro:property name="base_axel_offset" value="0.02" /><!-- Space btw top of beam and the each joint -->
+	<!-- <xacro:property name="base_axel_offset" value="0.02" />Space btw top of beam and the each joint -->
 	<!-- Frame -->
 	<xacro:property name="frame" value="frame" />

Commit message: fix: rear wheels were rotating in the wrong direction

File: src/pandora_description/urdf/leg.xacro (robot description, xacro)
@@ -182,5 +182,17 @@
 	<joint name="joint_${fork}_${wheel}_${leg_num}" type="continuous">
 		<origin xyz="0 0 ${wheel_radius + 0.015}" rpy="${PI/2} 0 0"/>
-		<axis xyz="0 0 1 "/>
+		<!-- Fix (2026-08-25): legs 3/4 are a front-to-back mirror of legs 1/2
+		     (see the base_link->frame joint's rpy sign flip above and the
+		     outer rotz=PI passed for legs 3/4 in pandora.xacro), so the same
+		     local "0 0 1" axis ends up pointing the opposite way in world
+		     frame for the rear wheels. Without this flip, velocity_controller
+		     driving all 4 wheels with the same-sign command spun the front
+		     and rear wheels in opposite directions (confirmed visually). -->
+		<xacro:if value="${leg_num == 1 or leg_num == 2}">
+			<axis xyz="0 0 1"/>
+		</xacro:if>
+		<xacro:if value="${leg_num == 3 or leg_num == 4}">
+			<axis xyz="0 0 -1"/>
+		</xacro:if>
 		<limit effort="350" velocity="20.0"/>
 	    <parent link="${fork}_${leg_num}"/>

Commit message: fix: namespace correctly assigned

File: src/pandora_description/urdf/leg.xacro (robot description, xacro)
@@ -186,5 +186,5 @@
 		     outer rotz=PI passed for legs 3/4 in pandora.xacro), so the same
 		     local "0 0 1" axis ends up pointing the opposite way in world
-		     frame for the rear wheels. Without this flip, velocity_controller
+		     frame for the rear wheels. Without this flip, wheel_controller
 		     driving all 4 wheels with the same-sign command spun the front
 		     and rear wheels in opposite directions (confirmed visually). -->
@@ -278,4 +278,16 @@
 			<state_interface name="velocity"/>
 		</joint>
+		<!-- Fix (2026-08-25): passive joint, like frame_rocker above; its
+		     actual angle is dictated by the 4-bar loop closure (the
+		     gz-sim-detachable-joint-system plugin welding dummy_link_N to
+		     rocker_N in physics), not by any command_interface here. Without
+		     a state_interface, joint_state_broadcaster never published this
+		     joint's angle to /joint_states, so robot_state_publisher kept
+		     dummy_link_N's TF frozen at the URDF default instead of tracking
+		     the real physics-driven pose. -->
+		<joint name="joint_${coupler}_dummy_link_${leg_num}">
+			<state_interface name="position"/>
+			<state_interface name="velocity"/>
+		</joint>
 		<joint name="joint_${fork}_${wheel}_${leg_num}">
 			<command_interface name="velocity"/>
